File: encoder.sch (KiCad schematic (older format))
At the start: 11 parts, among them IC1 AS5048

Commit message: Add panelized PCB data
Parts:
- C1: footprint generic:generic-SMD1608 -> generic:generic-SMD2012; Fieldname (none) -> Value
Changed lines of the file:
@@
 LIBS:con-hirose
 LIBS:v-reg
+LIBS:projectionball_encoder_v1.00-cache
 EELAYER 25 0
 EELAYER END
@@
 encoding utf-8
 Sheet 1 1
-Title "Encoder Board For AS5048A, AS5047D with SPI"
-Date "2017-01-22"
-Rev "V1.2"
-Comp "Crescent"
+Title ""
+Date ""
+Rev ""
+Comp ""
 Comment1 ""
 Comment2 ""
@@
 F 0 "C1" H 8720 4260 50  0000 R TNN
 F 1 "10uF/CAPACITOR1608" H 8720 4190 50  0000 R TNN
-F 2 "generic:generic-SMD1608" H 8730 4400 20  0001 C CNN
+F 2 "generic:generic-SMD2012" H 8730 4400 20  0001 C CNN
 F 3 "" H 8700 4250 60  0000 C CNN
+F 4 "Value" H 8700 4250 60  0001 C CNN "Fieldname"
 	1    8700 4250
 	1    0    0    -1
